File: PCB/EagleFiles/ESP32C-Mini-MQL-Injection-V2.brd (EAGLE design)
At the start: 52.7 x 37.5 mm, 21 parts

Commit message: Updated traces
Routing:
- net GND: track 79.1 -> 79.6 mm
- net SDA: track 16.6 -> 16.0 mm
- net SW: track 7.77 -> 7.26 mm
- net A: track 6.51 -> 6.01 mm
Changed lines of the file:
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@@
 <vertex x="52.705" y="0"/>
 </polygon>
-<wire x1="12.065" y1="15.23" x2="7.62" y2="15.23" width="0.4064" layer="16"/>
+<wire x1="12.573" y1="15.23" x2="7.62" y2="15.23" width="0.4064" layer="16"/>
 <wire x1="7.62" y1="15.23" x2="8.89" y2="15.24" width="0.4064" layer="16"/>
 <contactref element="R5" pad="2"/>
@@
 <contactref element="U$5" pad="3V3"/>
 <contactref element="U$1" pad="P$1"/>
-<wire x1="10.033" y1="14.21" x2="11.335" y2="12.795" width="1.016" layer="16"/>
+<wire x1="10.16" y1="14.21" x2="11.335" y2="12.795" width="1.016" layer="16"/>
 <wire x1="11.335" y1="12.795" x2="15.875" y2="8.255" width="1.016" layer="16"/>
 <wire x1="15.875" y1="8.255" x2="18.415" y2="8.255" width="1.016" layer="16"/>
@@
 <contactref element="U$1" pad="P$3"/>
 <wire x1="18.415" y1="10.795" x2="17.78" y2="10.795" width="0.4064" layer="16"/>
-<wire x1="10.033" y1="16.25" x2="12.96" y2="16.25" width="0.4064" layer="16"/>
+<wire x1="10.16" y1="16.25" x2="12.96" y2="16.25" width="0.4064" layer="16"/>
 <wire x1="12.96" y1="16.25" x2="13.335" y2="15.875" width="0.4064" layer="16"/>
 <wire x1="13.335" y1="15.875" x2="13.335" y2="13.335" width="0.4064" layer="16"/>
@@
 <contactref element="U$5" pad="D3"/>
 <contactref element="U$1" pad="P$4"/>
-<wire x1="12.065" y1="17.27" x2="13.845" y2="17.27" width="0.6096" layer="16"/>
+<wire x1="12.573" y1="17.27" x2="13.845" y2="17.27" width="0.6096" layer="16"/>
 <wire x1="13.845" y1="17.27" x2="14.605" y2="16.51" width="0.6096" layer="16"/>
 <wire x1="14.605" y1="16.51" x2="14.605" y2="14.605" width="0.6096" layer="16"/>
@@
 <contactref element="U$5" pad="D2"/>
 <contactref element="U$1" pad="P$6"/>
-<wire x1="12.065" y1="19.31" x2="13.71" y2="19.31" width="0.6096" layer="16"/>
+<wire x1="12.573" y1="19.31" x2="13.71" y2="19.31" width="0.6096" layer="16"/>
 <wire x1="13.71" y1="19.31" x2="17.145" y2="15.875" width="0.6096" layer="16"/>
 <wire x1="17.145" y1="15.875" x2="18.415" y2="15.875" width="0.6096" layer="16"/>
@@
 <contactref element="U$5" pad="D1"/>
 <contactref element="U$1" pad="P$7"/>
-<wire x1="10.033" y1="20.33" x2="15.23" y2="20.33" width="0.4064" layer="16"/>
+<wire x1="10.16" y1="20.33" x2="15.23" y2="20.33" width="0.4064" layer="16"/>
 <wire x1="15.23" y1="20.33" x2="17.145" y2="18.415" width="0.4064" layer="16"/>
 <wire x1="17.145" y1="18.415" x2="18.415" y2="18.415" width="0.4064" layer="16"/>
@@
 <contactref element="U$5" pad="D0"/>
 <contactref element="U$1" pad="P$8"/>
-<wire x1="12.065" y1="21.35" x2="18.02" y2="21.35" width="0.6096" layer="16"/>
+<wire x1="12.573" y1="21.35" x2="18.02" y2="21.35" width="0.6096" layer="16"/>
 <wire x1="18.02" y1="21.35" x2="18.415" y2="20.955" width="0.6096" layer="16"/>
 </signal>
