File: PCB/EagleFiles/ESP32C-Mini-MQL-Injection-V2.sch (EAGLE design)
At the start: 21 parts

Commit message: Updated traces
Other:
- note added: "Modifications for next build: none"
- note removed: "Modifications for next build: - GPIO9 is used for boot mode and connected to USB DTR, don't use"
Changed lines of the file:
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@@
 Minimal Quantity Lubrication
 Injection system</text>
-<text x="-66.04" y="53.34" size="2.54" layer="97">Modifications for next build:
-- GPIO9 is used for boot mode and connected to USB DTR, don't use
-</text>
+<text x="-66.04" y="53.34" size="2.54" layer="97">Modifications for next build: none</text>
 </plain>
 <instances>
