File: PCB/EagleFiles/RotaryEncoder.sch (EAGLE design)
At the start: 2 parts, among them SW1 ROTARY-ENCODER

Commit message: Updated traces
Connections:
- net A: now also SW1R.C; no longer SW1R.A
- net B: now also SW1R.A; no longer SW1R.C
Changed lines of the file:
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@@
 </segment>
 <segment>
-<pinref part="SW1" gate="R" pin="C"/>
-<wire x1="99.06" y1="58.42" x2="104.14" y2="58.42" width="0.1524" layer="91"/>
-<label x="104.14" y="58.42" size="1.778" layer="95"/>
+<pinref part="SW1" gate="R" pin="A"/>
+<wire x1="99.06" y1="53.34" x2="104.14" y2="53.34" width="0.1524" layer="91"/>
+<label x="104.14" y="53.34" size="1.778" layer="95"/>
 </segment>
 </net>
@@
 </segment>
 <segment>
-<pinref part="SW1" gate="R" pin="A"/>
-<wire x1="99.06" y1="53.34" x2="104.14" y2="53.34" width="0.1524" layer="91"/>
-<label x="104.14" y="53.34" size="1.778" layer="95"/>
+<pinref part="SW1" gate="R" pin="C"/>
+<wire x1="99.06" y1="58.42" x2="104.14" y2="58.42" width="0.1524" layer="91"/>
+<label x="104.14" y="58.42" size="1.778" layer="95"/>
 </segment>
 </net>
